File: Schematics/Block-Party/Block-Party.kicad_sch (KiCad schematic)
At the start: 10 parts

Commit message: Created block party main board schematic
Other:
- company: (none) -> Block Party
- title: (none) -> Bottom PCB Schematic
Changed lines of the file:
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@@
 (kicad_sch (version 20230121) (generator eeschema)
   (paper "A4")
+  (title_block
+    (title "Bottom PCB Schematic")
+    (date "2024-02-10")
+    (rev "1.0.0")
+    (company "Block Party")
+  )
   (no_connect (at 158.75 102.87))
   (wire (pts (xy 166.37 88.9) (xy 160.02 88.9))
