File: Schematics/Block-Party/Block-Party-Cube-Bottom-Board/Block-Party-Bottom-Board.kicad_sch (KiCad schematic)
At the start: 10 parts

Commit message: Revision 1.01 of the PCBs
Parts:
- removed J1, J2, J3, J4: ~, Connector_PinHeader_2.54mm:PinHeader_1x01_P2.54mm_Vertical, symbol Quinn_lib:HDR-M-2.54_1x1
- added J6: YTC-A1001LF-04A, adafruit-jst-4328:ADAFRUIT_4328, symbol 4328:4328
- added TP1: Diode5V, TestPoint:TestPoint_Pad_D1.0mm, symbol Connector:TestPoint
- added TP2: DODI, TestPoint:TestPoint_Pad_D1.0mm, symbol Connector:TestPoint
- added TP4: DO, TestPoint:TestPoint_Pad_D1.0mm, symbol Connector:TestPoint
- added TP5: 5V, TestPoint:TestPoint_Pad_D1.0mm, symbol Connector:TestPoint
- added TP6: DI, TestPoint:TestPoint_Pad_D1.0mm, symbol Connector:TestPoint
- C1: MANUFACTURER (none) -> Samwha Capacitor; Manufacturer_Part_Number (none) -> CS2012X5R475K500NRE
- J5: now not fitted; now left out of the parts list
- LED1, LED2: MANUFACTURER (none) -> XINGLIGHT; Manufacturer_Part_Number (none) -> XL-1615RGBC-RF
- R1: MANUFACTURER (none) -> YAGEO; Manufacturer_Part_Number (none) -> AC0805FR-0710KL
Connections:
- net +5V: now also J6.4, TP5.1
- net D5V: now also TP1.1
- net DIN: now also TP6.1
- net DOUT: now also J6.3, TP4.1
- net GND: now also J6.1, J6.SH1 (SHIELD), J6.SH2 (SHIELD)
- net SENSE: now also J6.2
- net at LED1.4 (DI), LED2.1 (DO): now also TP2.1

Commit message: Found a good jst part number and updated the BOMs
Parts:
- J6: value YTC-A1001LF-04A -> BM04B-SRSS-TB; MANUFACTURER YIYUAN -> JST; Manufacturer_Part_Number YTC-A1001LF-04A -> BM04B-SRSS-TB
Changed lines of the file:
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@@
 			)
 		)
-		(property "Value" "YTC-A1001LF-04A"
+		(property "Value" "BM04B-SRSS-TB"
 			(at 135.89 123.19 0)
 			(effects
@@
 			)
 		)
-		(property "MANUFACTURER" "YIYUAN"
+		(property "MANUFACTURER" "JST"
 			(at 135.89 133.35 0)
 			(effects
@@
 			)
 		)
-		(property "Manufacturer_Part_Number" "YTC-A1001LF-04A"
+		(property "Manufacturer_Part_Number" "BM04B-SRSS-TB"
 			(at 135.89 133.35 0)
 			(effects

Commit message: Updated micro configuration files to match the new micro we're using.
Parts:
- LED1, LED2: Manufacturer_Part_Number XL-1615RGBC-RF -> XINGLIGHT XL-1615RGBC-WS2812B
Changed lines of the file:
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@@
 			)
 		)
-		(property "Manufacturer_Part_Number" "XL-1615RGBC-RF"
+		(property "Manufacturer_Part_Number" "XINGLIGHT XL-1615RGBC-WS2812B"
 			(at 172.72 85.09 0)
 			(effects
@@
 			)
 		)
-		(property "Manufacturer_Part_Number" "XL-1615RGBC-RF"
-			(at 144.78 85.09 0)
-			(effects
+		(property "Manufacturer_Part_Number" "XINGLIGHT XL-1615RGBC-WS2812B"
+			(at 144.78 85.09 0)
+			(effects
